File: OrientationTest.kicad_sch (KiCad schematic)
At the start: 2 parts

Commit message: asdf
Connections:
- net at Q?.2 (C): now also R?.2
Other:
- moved on the sheet: Q?, R?
Changed lines of the file:
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@@
 (kicad_sch (version 20211123) (generator eeschema)
   (paper "A4")
-  (symbol (lib_id "Device:Q_NPN_BCE") (at 167.64 95.25 0) (unit 1)
+  (junction (at 165.1 68.58) (diameter 0) (color 0 0 0 0)
+  )
+  (junction (at 149.86 80.01) (diameter 0) (color 0 0 0 0)
+  )
+  (wire (pts (xy 156.21 80.01) (xy 156.21 68.58))
+    (stroke (width 0) (type default) (color 0 0 0 0))
+  )
+  (wire (pts (xy 165.1 60.96) (xy 165.1 68.58))
+    (stroke (width 0) (type default) (color 0 0 0 0))
+  )
+  (wire (pts (xy 149.86 80.01) (xy 156.21 80.01))
+    (stroke (width 0) (type default) (color 0 0 0 0))
+  )
+  (wire (pts (xy 156.21 68.58) (xy 165.1 68.58))
+    (stroke (width 0) (type default) (color 0 0 0 0))
+  )
+  (wire (pts (xy 149.86 80.01) (xy 149.86 64.135))
+    (stroke (width 0) (type default) (color 0 0 0 0))
+  )
+  (wire (pts (xy 127 60.96) (xy 165.1 60.96))
+    (stroke (width 0) (type default) (color 0 0 0 0))
+  )
+  (wire (pts (xy 143.51 91.44) (xy 143.51 80.01))
+    (stroke (width 0) (type default) (color 0 0 0 0))
+  )
+  (wire (pts (xy 139.065 64.135) (xy 139.065 67.945))
+    (stroke (width 0) (type default) (color 0 0 0 0))
+  )
+  (wire (pts (xy 149.86 64.135) (xy 139.065 64.135))
+    (stroke (width 0) (type default) (color 0 0 0 0))
+  )
+  (wire (pts (xy 173.99 68.58) (xy 173.99 86.36))
+    (stroke (width 0) (type default) (color 0 0 0 0))
+  )
+  (wire (pts (xy 143.51 80.01) (xy 149.86 80.01))
+    (stroke (width 0) (type default) (color 0 0 0 0))
+  )
+  (wire (pts (xy 165.1 68.58) (xy 173.99 68.58))
+    (stroke (width 0) (type default) (color 0 0 0 0))
+  )
+  (label "ALABEL" (at 217.17 92.71 0)
+    (effects (font (size 1.27 1.27)) (justify left bottom))
+  )
+  (label "ALABEL" (at 180.34 82.55 0)
+    (effects (font (size 1.27 1.27)) (justify left bottom))
+  )
+  (label "ALABEL" (at 205.74 77.47 0)
+    (effects (font (size 1.27 1.27)) (justify left bottom))
+  )
+  (label "ALABEL" (at 214.63 85.09 0)
+    (effects (font (size 1.27 1.27)) (justify left bottom))
+  )
+  (label "ALABEL" (at 198.12 86.36 0)
+    (effects (font (size 1.27 1.27)) (justify left bottom))
+  )
+  (label "ALABEL" (at 203.2 105.41 0)
+    (effects (font (size 1.27 1.27)) (justify left bottom))
+  )
+  (label "ALABEL" (at 193.04 68.58 0)
+    (effects (font (size 1.27 1.27)) (justify left bottom))
+  )
+  (label "ALABEL" (at 200.66 59.69 0)
+    (effects (font (size 1.27 1.27)) (justify left bottom))
+  )
+  (symbol (lib_id "Device:Q_NPN_BCE") (at 171.45 91.44 0) (unit 1)
     (in_bom yes) (on_board yes)
-    (property "Reference" "Q?" (id 0) (at 172.72 93.98 0)
+    (property "Reference" "Q?" (id 0) (at 176.53 90.17 0)
       (effects (font (size 1.27 1.27)) (justify left))
     )
-    (property "Value" "Q_NPN_BCE" (id 1) (at 172.72 96.52 0)
+    (property "Value" "Q_NPN_BCE" (id 1) (at 176.53 92.71 0)
       (effects (font (size 1.27 1.27)) (justify left))
     )
-    (property "Footprint" "" (id 2) (at 172.72 92.71 0)
+    (property "Footprint" "" (id 2) (at 176.53 88.9 0)
       (effects (font (size 1.27 1.27)) hide)
     )
-    (property "Datasheet" "~" (id 3) (at 167.64 95.25 0)
+    (property "Datasheet" "~" (id 3) (at 171.45 91.44 0)
       (effects (font (size 1.27 1.27)) hide)
     )
@@
     (pin "3")
   )
-  (symbol (lib_id "Device:R_US") (at 143.51 95.25 90) (unit 1)
+  (symbol (lib_id "Device:R_US") (at 143.51 95.25 180) (unit 1)
     (in_bom yes) (on_board yes)
-    (property "Reference" "R?" (id 0) (at 143.51 92.71 90))
-    (property "Value" "R_US" (id 1) (at 143.51 97.79 90))
-    (property "Footprint" "" (id 2) (at 143.764 94.234 90)
+    (property "Reference" "R?" (id 0) (at 140.97 95.25 90))
+    (property "Value" "R_US" (id 1) (at 146.05 95.25 90))
+    (property "Footprint" "" (id 2) (at 142.494 94.996 90)
       (effects (font (size 1.27 1.27)) hide)
     )
