File: OrientationTest.kicad_sch (KiCad schematic)
At the start: 2 parts

Commit message: aoiweur
Connections:
- no-connect marks 0 -> 1
Other:
- note added: "Some Text"
Changed lines of the file:
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@@
   (junction (at 149.86 80.01) (diameter 0) (color 0 0 0 0)
   )
+  (no_connect (at 188.595 57.785))
   (wire (pts (xy 156.21 80.01) (xy 156.21 68.58))
     (stroke (width 0) (type default) (color 0 0 0 0))
@@
     (stroke (width 0) (type default) (color 0 0 0 0))
   )
+  (text "Some Text" (at 203.2 65.405 0)
+    (effects (font (size 1.27 1.27)) (justify left bottom))
+  )
   (label "ALABEL" (at 217.17 92.71 0)

Commit message: zlxkjf
Other:
- note added: "This is some multiline text"
Changed lines of the file:
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@@
+    (effects (font (size 1.27 1.27)) (justify left bottom))
+  )
+  (text "This is some\nmultiline text" (at 170.815 62.23 0)
     (effects (font (size 1.27 1.27)) (justify left bottom))
   )

Commit message: alskdfjk
Connections:
- net GLABEL: no longer Q?.2 (C), R?.2
Changed lines of the file:
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@@
 (kicad_sch (version 20211123) (generator eeschema)
   (paper "A4")
+  (junction (at 149.86 80.01) (diameter 0) (color 0 0 0 0)
+  )
   (junction (at 165.1 68.58) (diameter 0) (color 0 0 0 0)
   )
-  (junction (at 149.86 80.01) (diameter 0) (color 0 0 0 0)
+  (no_connect (at 188.595 57.785))
+  (bus_entry (at 192.405 86.995) (size 2.54 2.54)
+    (stroke (width 0) (type default) (color 0 0 0 0))
   )
-  (no_connect (at 188.595 57.785))
-  (wire (pts (xy 156.21 80.01) (xy 156.21 68.58))
+  (wire (pts (xy 165.1 68.58) (xy 173.99 68.58))
     (stroke (width 0) (type default) (color 0 0 0 0))
   )
@@
     (stroke (width 0) (type default) (color 0 0 0 0))
   )
+  (bus (pts (xy 192.405 86.995) (xy 192.405 91.44))
+    (stroke (width 0) (type default) (color 0 0 0 0))
+  )
+  (bus (pts (xy 192.405 73.66) (xy 192.405 86.995))
+    (stroke (width 0) (type default) (color 0 0 0 0))
+  )
   (wire (pts (xy 149.86 80.01) (xy 149.86 64.135))
     (stroke (width 0) (type default) (color 0 0 0 0))
@@
     (stroke (width 0) (type default) (color 0 0 0 0))
   )
-  (wire (pts (xy 139.065 64.135) (xy 139.065 67.945))
+  (wire (pts (xy 163.83 96.52) (xy 173.99 96.52))
     (stroke (width 0) (type default) (color 0 0 0 0))
   )
-  (wire (pts (xy 149.86 64.135) (xy 139.065 64.135))
-    (stroke (width 0) (type default) (color 0 0 0 0))
-  )
-  (wire (pts (xy 173.99 68.58) (xy 173.99 86.36))
+  (wire (pts (xy 153.67 67.945) (xy 139.065 67.945))
     (stroke (width 0) (type default) (color 0 0 0 0))
   )
@@
     (stroke (width 0) (type default) (color 0 0 0 0))
   )
-  (wire (pts (xy 165.1 68.58) (xy 173.99 68.58))
-    (stroke (width 0) (type default) (color 0 0 0 0))
-  )
   (text "Some Text" (at 203.2 65.405 0)
     (effects (font (size 1.27 1.27)) (justify left bottom))
   )
-  (text "This is some\nmultiline text" (at 170.815 62.23 0)
+  (text "This is some\nmultiline text" (at 170.815 62.23 90)
     (effects (font (size 1.27 1.27)) (justify left bottom))
   )
